File: PCB/galwo.kicad_sch (KiCad schematic)
At the start: 20 parts, among them J1 Conn_02x20_Odd_Even, J2 Screw_Terminal_01x02, J3 Screw_Terminal_01x02, J4 Screw_Terminal_01x02, J5 Screw_Terminal_01x02, J6 Screw_Terminal_01x02, J7 Screw_Terminal_01x02, P1 Conn_01x03, U1 MCP4922, U2 MCP4922, U3 MCP4922, U4 TL074, U5 TL074, U6 TL074, U7 TL074

Commit message: Add files via upload
Parts:
- removed C2, C3, C4: 100nF, Capacitor_THT:C_Disc_D3.8mm_W2.6mm_P2.50mm, symbol Device:C
- removed J1: Conn_02x20_Odd_Even, Connector_PinSocket_2.54mm:PinSocket_2x20_P2.54mm_Vertical, symbol Connector_Generic:Conn_02x20_Odd_Even
- removed J7: Screw_Terminal_01x02, TerminalBlock_Phoenix:TerminalBlock_Phoenix_MKDS-1,5-2-5.08_1x02_P5.08mm_Horizontal, symbol Connector:Screw_Terminal_01x02
- removed U2, U3: MCP4922, Package_DIP:DIP-14_W7.62mm, symbol Analog_DAC:MCP4922
- removed U4, U5, U6, U7: TL074, Package_DIP:DIP-14_W7.62mm, symbol Amplifier_Operational:TL074
- added A1: RaspberryPi_Pico_W, proba:RaspberryPi_Pico_W_SMD_HandSolder_tht, symbol MCU_Module:RaspberryPi_Pico_W
- added C1: 100nF, Capacitor_THT:C_Disc_D5.0mm_W2.5mm_P5.00mm, symbol Device:C
- added H1, H2, H3, H4: MountingHole, MountingHole:MountingHole_2.7mm_M2.5, symbol Mechanical:MountingHole
- added J1: Conn_01x02, TerminalBlock_Phoenix:TerminalBlock_Phoenix_MKDS-1,5-2-5.08_1x02_P5.08mm_Horizontal, symbol Connector_Generic:Conn_01x02
- added J7: Conn_02x02_Counter_Clockwise, proba:Bez_nazwy, symbol Connector_Generic:Conn_02x02_Counter_Clockwise
- added Q1, Q2, Q3: Q_NPN_BCE, Package_TO_SOT_THT:TO-92L_Inline, symbol Transistor_BJT:Q_NPN_BCE
- added R1, R2, R3: 1k, Resistor_THT:R_Axial_DIN0207_L6.3mm_D2.5mm_P7.62mm_Horizontal, symbol Device:R
- added U1: TL074, Package_DIP:DIP-14_W7.62mm, symbol Amplifier_Operational:TL074
- C2: renamed from C6; footprint Capacitor_THT:C_Disc_D3.8mm_W2.6mm_P2.50mm -> Capacitor_THT:C_Disc_D5.0mm_W2.5mm_P5.00mm
- C3: renamed from C5; footprint Capacitor_THT:C_Disc_D3.8mm_W2.6mm_P2.50mm -> Capacitor_THT:C_Disc_D5.0mm_W2.5mm_P5.00mm
- renumbered U1 to U2
Connections:
- net -15V: now also C3.1, P1.1 (Pin_1), U1.11 (V-)
- net GND: now also C2.1, C3.2, J2.2 (Pin_2), J3.2 (Pin_2), P1.2 (Pin_2), U2.12 (Vss), U2.8 (~{LDAC}), A1.13 (GND), A1.18 (GND), A1.23 (GND), A1.28 (GND), A1.3 (GND), A1.38 (GND), A1.8 (GND), C1.2, J1.2 (Pin_2), J7.1 (Pin_1), J7.4 (Pin_4), Q1.3 (E), Q2.3 (E), Q3.3 (E), U1.3 (+), U1.5 (+)
- net at J5.1 (Pin_1): now also Q3.2 (C)
- net at U2.1 (Vdd), U2.11 (VrefB), U2.13 (VrefA)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: now also A1.36 (3V3)
- net at U2.5 (SDI): now also A1.25 (GPIO19)
- net at U2.4 (SCK): now also A1.24 (GPIO18)
- net at U2.3 (~{CS}): now also A1.27 (GPIO21)
- net 15V: now reaches C2.2, P1.3 (Pin_3)
- net 15V: now also J7.2 (Pin_2), U1.4 (V+); no longer C3.2
- net at J6.1 (Pin_1): now also Q1.2 (C)
- net at J3.1 (Pin_1): now also U1.13 (-), U1.14
- net at U2.10 (VB): now also U1.12 (+)
- net at U2.14 (VA): now also U1.10 (+)
- net at J2.1 (Pin_1): now also U1.8, U1.9 (-)
- net at J4.1 (Pin_1): now also Q2.2 (C)
- new net: A1.39 (VSYS), C1.1, J1.1 (Pin_1), J4.2 (Pin_2), J5.2 (Pin_2), J6.2 (Pin_2), J7.3 (Pin_3)
- new net: A1.19 (GPIO14), R3.1
- new net: Q3.1 (B), R3.2
- new net: A1.17 (GPIO13), R2.1
- new net: A1.20 (GPIO15), R1.1
- new net: Q2.1 (B), R2.2
- new net: U1.1, U1.2 (-)
- new net: Q1.1 (B), R1.2
- new net: U1.6 (-), U1.7
- no-connect marks 0 -> 25
Other:
- note added: "+5"
- note added: "+5V Laser"
- note added: "B"
- note added: "G"
- note added: "GND"
- note added: "GND Laser"
- note added: "Os X"
- note added: "Os Y"
- note added: "R"
- moved on the sheet: C2, C3, U2
